File: Schematics/launchbox_launchBox/launchbox_launchBox.kicad_pcb (KiCad board)
At the start: 2 copper layers, 10 parts, among them J3 Msg_Recv_LED, J4 Rail_isArmed_LED, J7 Conn_01x04_Pin, SW1 Arm_switch, SW2 fire_btn, SW3 Batt_on_off

Commit message: completed launch box pcb
Parts:
- removed J7: Conn_01x04_Pin, Connector_PinHeader_2.54mm:PinHeader_1x04_P2.54mm_Vertical
- removed SW3: Batt_on_off, Connector_PinHeader_2.54mm:PinHeader_1x02_P2.54mm_Vertical
- added BZ1: Buzzer, Connector_PinHeader_2.54mm:PinHeader_1x02_P2.54mm_Vertical, F.Cu at (121.9, 100.3)
- added D1: LED, Connector_PinHeader_2.54mm:PinHeader_1x02_P2.54mm_Vertical, F.Cu at (121.9, 92.7)
- added H1: MountingHole_Pad, MountingHole:MountingHole_3.2mm_M3_Pad_TopBottom, F.Cu at (152.4, 63.5)
- added H2: MountingHole_Pad, MountingHole:MountingHole_3.2mm_M3_Pad_TopBottom, F.Cu at (120.7, 63.5)
- added H3: MountingHole_Pad, MountingHole:MountingHole_3.2mm_M3_Pad_TopBottom, F.Cu at (120.7, 108.0)
- added H4: MountingHole_Pad, MountingHole:MountingHole_3.2mm_M3_Pad_TopBottom, F.Cu at (152.4, 108.0)
- added J1: batt_switched_pwr, Connector_PinHeader_2.54mm:PinHeader_1x02_P2.54mm_Vertical, F.Cu at (149.9, 69.8)
- added J2: Msg_Recv_LED, Connector_PinHeader_2.54mm:PinHeader_1x02_P2.54mm_Vertical, F.Cu at (121.9, 85.1)
- J3: value Msg_Recv_LED -> Rail_isArmed_LED
- J4: value Rail_isArmed_LED -> Conn_01x04_Pin; footprint Connector_PinHeader_2.54mm:PinHeader_1x02_P2.54mm_Vertical -> Connector_PinHeader_2.54mm:PinHeader_1x04_P2.54mm_Vertical
- R1, R2, R3: moved to B.Cu
- moved SW1 61.3 mm to (147.3, 97.8), turned to 180 degrees
- moved A1 61.0 mm to (127.0, 67.3)
- moved J4 59.4 mm to (147.3, 82.5), turned to 180 degrees
- moved SW2 53.6 mm to (147.3, 90.2), turned to 180 degrees
- moved R1 44.8 mm to (130.8, 91.1), turned to 90 degrees
- moved R2 41.6 mm to (130.8, 83.5), turned to 90 degrees
- moved R3 40.7 mm to (130.8, 77.1), turned to -90 degrees
- moved J3 38.0 mm to (121.9, 77.5), turned to 180 degrees
Connections:
- A1 pad 1: unconnected-(A1-D1/TX-Pad1) -> /nano_to_rad
- A1 pad 2: unconnected-(A1-D0/RX-Pad2) -> /rad_to_nano
- A1 pad 27: Net-(A1-+5V) -> +5V
- A1 pad 30: Net-(A1-VIN) -> VIN
- J3 pad 1: Net-(J3-Pin_1) -> GND
- J3 pad 2: GND -> Net-(J3-Pin_1)
- J4 pad 1: Net-(J4-Pin_1) -> GND
- J4 pad 2: GND -> +5V
- R2 pad 1: Net-(J3-Pin_1) -> Net-(J2-Pin_1)
- R3 pad 1: Net-(J4-Pin_1) -> Net-(J3-Pin_1)
- SW1 pad 1: Net-(A1-+5V) -> +5V
- SW1 pad 2: Net-(A1-+5V) -> Net-(A1-A1)
Routing:
- net /nano_to_rad: track 0.00 -> 30.1 mm
- net +5V: track 0.00 -> 27.8 mm
- net /trigger_pin: track 0.00 -> 23.5 mm
- net /rad_to_nano: track 0.00 -> 22.4 mm
- net Net-(A1-A1): track 0.00 -> 17.3 mm
- net Net-(BZ1-+): track 0.00 -> 11.3 mm
- net Net-(J2-Pin_1): track 0.00 -> 9.65 mm
- net Net-(J3-Pin_1): track 0.00 -> 9.42 mm
- net /rail_continuity_LED_PIN: track 0.00 -> 7.18 mm
- net VIN: track 0.00 -> 6.13 mm
- net /rail_isArmed_LED_pin: track 0.00 -> 4.04 mm
- net Net-(A1-D7): track 0.00 -> 3.81 mm
- net /msg_recv_LED_pin: track 0.00 -> 3.81 mm
- added copper zone on F.Cu, net GND
Other:
- board outline added: 40.8 x 52.1 mm
- board text added: "armed"
- board text added: "buzz+"
- board text added: "cont+"
- board text added: "data+"
- board text added: "gnd"
- board text added: "launch"
- board text added: "nano2rad"
- board text added: "nano_5v"
- board text added: "rad2nano"
- board text added: "rad_5v"
- board text added: "rad_gnd"
- board text added: "rail arm+"
- board text added: "vin+"
