File: Schematics/launchbox_launchBox/launchbox_launchBox.kicad_pcb (KiCad board)
At the start: 2 copper layers, 40.8 x 52.1 mm, 16 parts, among them J1 batt_switched_pwr, J2 Msg_Recv_LED, J3 Rail_isArmed_LED, J4 Conn_01x04_Pin, SW1 Arm_switch, SW2 fire_btn

Commit message: Added version, title, and PR logo to LCU
Parts:
- added G***: LOGO, logo:Logo, B.Cu at (135.0, 101.0)
Other:
- board text added: "Launch Control Unit v1.1.0"
